File: 3 Realization/Schematic/DDS Tone Shield/DDS Tone Shield.sch (EAGLE design)
At the start: 32 parts

Commit message: Layout changes again
Layout changes again
Parts:
- removed FRAME1: FRAME-LETTERNO_PACKAGE, DDS Tone Shield:FRAME-LETTERNO_PACKAGE
- removed J2, J3, J4: (no value), DDS Tone Shield:CONN_04
- removed J5: (no value), DDS Tone Shield:CONN_02
- removed LED1: (no value), DDS Tone Shield:LED1206
- removed U$1, U$2, U$3, U$4, U$5: (no value), DDS Tone Shield:POT1
- added D1: BLUE, DDS Tone Shield:LED-BLUE1206
- added FRAME2: FRAME-LEDGER, 1-Generic:FRAME-LEDGER
- added L1, L2: 4.7mH, DDS Tone Shield:INDUCTOR
- added R10: 100kohm, DDS Tone Shield:POT2
- added R11: 5kohm, DDS Tone Shield:POT1
- added R12, R13, R14: 10kohm, DDS Tone Shield:POT1
- added R7: 3.9kohm, DDS Tone Shield:RESISTOR1206
- added R8: 5.6kohm, DDS Tone Shield:RESISTOR1206
- added U$9: (no value), DDS Tone Shield:SPEAKER
- added U2: ATTINY85-20P, DDS Tone Shield:ATTINY85-20P
- added U3: LM386N, DDS Tone Shield:LM386
- C1, C2, C4: value (none) -> 100nF; device 1-Generic:CAP_POL1206 -> DDS Tone Shield:CAP_POL1206
- C3, C5: value (none) -> 47nF; device 1-Generic:CAP_POL1206 -> DDS Tone Shield:CAP_POL1206
- C6, C7, C8, C9: value 4.7uF -> 22nF; device DDS Tone Shield:4.7UF-1206-16V-(+80/-20%) -> DDS Tone Shield:CAP_POL1206
- J1: device DDS Tone Shield:CONN_04 -> DDS Tone Shield:CONN_02
- R1: value (none) -> 330ohm
- R2, R3: value (none) -> 270ohm
- R4, R6: value (none) -> 1kohm
- R5: value (none) -> 3.9kohm
- R9: value (none) -> 5kohm; device DDS Tone Shield:RESISTOR1206 -> DDS Tone Shield:POT1
- S1: value DIP-04SMD -> PUSHBUTTON; device DDS Tone Shield:DIP-04SMD -> DDS Tone Shield:PUSHBUTTON
- S2: value PUSHBUTTON -> DIP-04SMD; device DDS Tone Shield:PUSHBUTTON -> DDS Tone Shield:DIP-04SMD
- U1: device 1-Generic:ARDUINO_SHIELD -> DDS Tone Shield:ARDUINO_SHIELD
Connections:
- removed net +IN: J3.2
- removed net -IN: J3.3, R4.2, S3.O, U$4.E
- removed net BYPASS: J4.3
- removed net GAIN: J3.4, J4.4
- removed net N$12: U$2.S
- removed net N$2: C2.+, R5.2, U$1.E
- removed net N$3: C4.+, C5.+, R2.2
- removed net N$5: C3.-, R9.2, U$2.E
- removed net N$6: C5.-, R3.2, U$5.E
- removed net N$7: C3.+, R2.1, R5.1, S3.S
- removed net N$8: R4.1, U$1.S, U$5.S
- removed net PB0: J1.1, U1.D11
- removed net PB1: J1.2, LED1.A, R6.2, S2.B1, S2.B2, U1.D12
- removed net PB2: J1.3, U$3.S, U1.D13
- removed net PB3: J2.3, S1.1B, S1.2B, S1.3B, S1.4B
- removed net PB4: J2.2, R1.1
- removed net PB5: J2.4, U1.D10
- removed net TONE: C1.+, R1.2, S3.P
- removed net TONE_DIP1: S1.1A, U1.D9
- removed net TONE_DIP2: S1.2A, U1.D6
- removed net TONE_DIP3: S1.3A, U1.D5
- removed net TONE_DIP4: S1.4A, U1.D3
- removed net VCC: C6.1, C7.1, C8.1, C9.1, J1.4, S2.A1, S2.A2, U$3.E, U1.5V
- removed net VOUT: J4.1, J5.2, U$4.S
- removed net VSS: J4.2
- new net +5V: C1.+, C2.-, R9.E, S1.A1, S1.A2, U1.5V, U2.VCC, U3.V+
- new net 3BAND_SIGNAL_OUT: R12.S, R13.S, R14.S, R8.1
- new net ATTINY_[PROGRAM_SIGNAL_1: U1.D10, U2.NRES/PB5
- new net ATTINY_[PROGRAM_SIGNAL_2: U1.D11, U2.PB0
- new net CHEBYSHEV_OUT: R10.S, S3.P
- new net DDS_TONE_OUTPUT_SIGNAL: R2.1, U2.PB4
- new net N$13: C3.+, L1.P$1, R2.2
- new net N$14: C4.+, L1.P$2, L2.P$1
- new net N$15: C5.+, L2.P$2, R10.E, R3.1
- new net N$17: R11.E, R8.2, S3.O, U3.-IN
- new net N$18: C6.-, R12.E, R4.1
- new net N$19: C7.+, R13.E, R5.2
- new net N$20: C8.-, R6.1, R7.1
- new net N$21: C9.+, R14.E, R7.2
- new net N$26: C6.+, C8.+, R5.1, S3.S
- new net ON_OFF_STATE_SIGNAL: D1.A, R1.2, S1.B1, S1.B2, U1.D12, U2.PB1
- new net SPEAKER_SIGNAL_IN: J1.1, R11.S, U3.OUT
- new net UNO_TONE_SIGNAL_1: S2.1A, U1.D3
- new net UNO_TONE_SIGNAL_2: S2.2A, U1.D5
- new net UNO_TONE_SIGNAL_3: S2.3A, U1.D6
- new net UNO_TONE_SIGNAL_4: S2.4A, U1.D9
- new net UNO_TONE_SIGNAL_MASTER: S2.1B, S2.2B, S2.3B, S2.4B, U2.PB3
- new net VAR_FREQ_SIGNAL: R9.S, U1.D13, U2.PB2
- net GND: now also C2.+, C3.-, C5.-, C7.-, C9.-, D1.C, J1.2, R1.1, R10.A, R11.A, R12.A, R13.A, R14.A, R3.2, R4.2, R6.2, R9.A, U2.GND, U3.+IN, U3.V-; no longer C2.-, C6.2, C7.2, C8.2, C9.2, J2.1, J3.1, J5.1, LED1.C, R3.1, R6.1, R9.1, U$1.A, U$2.A, U$3.A, U$4.A, U$5.A
Other:
- note added: "Zacher Tiburzi"
- moved on the sheet: C1, C2, C3, C4, C5, R1, R2, R3, R4, R5, R6, S3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
