File: 3 Realization/Eagle/DDS Tone Shield/DDS Tone Shield.brd (EAGLE design)
At the start: 55.1 x 177.8 mm, 37 parts, among them J1 Speaker Header, U2 ATTINY85-20P, U3 LM386N

Commit message: layout
layout
Parts:
- removed C1, C2, C4: 100nF, DDS Tone Shield:EIA3216
- removed C3, C5: 47nF, DDS Tone Shield:EIA3216
- removed C6, C7, C8, C9: 22nF, DDS Tone Shield:EIA3216
- removed D1: BLUE, DDS Tone Shield:LED-1206
- removed J1: Speaker Header, DDS Tone Shield:1X02
- removed R10: 100kohm, DDS Tone Shield:5150500311
- removed S1: PUSHBUTTON, DDS Tone Shield:3CSH9_MEC_PUSHBUTTON
- removed S2: DIP-04SMD, DDS Tone Shield:DIPSWITCH-04-SMD
- removed S3: Slide Switch, DDS Tone Shield:JS102011SAQN
- removed U1: (no value), DDS Tone Shield:DUEMILANOVE_SHIELD
- added C11, C13: 47nF, 1-Generic:EIA3216
- added C12, C18: 100nF, 1-Generic:EIA3216
- added C14, C15, C16, C17: 22nF, 1-Generic:EIA3216
- added JP1: Arduino jumpers, DDS Tone Shield:DUEMILANOVE_SHIELD
- added JP10, JP11, JP3, JP4, JP5, JP6, JP7, JP8, JP9: JUMPER-SMT_2_NC_PASTE_SILK, DDS Tone Shield:SMT-JUMPER_2_NC_PASTE_SILK
- added JP2: Speaker Header, DDS Tone Shield:1X02
- added LED1: BLUE, DDS Tone Shield:LED-1206
- added R16, R17: 2200, DDS Tone Shield:1206
- added R24: 270ohm, DDS Tone Shield:1206
- added R29: 100k, DDS Tone Shield:RK09K/RK09D_SERIES
- added SW1: PUSHBUTTON, DDS Tone Shield:3CSH9_MEC_PUSHBUTTON
- added SW2: DIP-04SMD, DDS Tone Shield:DIPSWITCH-04-SMD
- added SW3: Slide Switch, DDS Tone Shield:JS102011SAQN
- C10: value (none) -> 100nF; device DDS Tone Shield:EIA3216 -> 1-Generic:EIA3216
- R1: value 330ohm -> 10kohm
- R8: value 5.6kohm -> 2200
- Y1: value (none) -> Speaker
- moved FRAME2 108.5 mm to (0.20, 146.8)
- moved C10 44.6 mm to (20.5, 43.2), turned to 270 degrees
- moved R15 28.9 mm to (27.6, 3.22), turned to 180 degrees
- moved R3 27.5 mm to (34.1, 18.5), turned to 0 degrees
- moved L4 21.4 mm to (27.0, 24.0)
- moved R2 20.6 mm to (26.7, 39.1)
- moved L3 20.1 mm to (27.0, 33.0)
- moved R1 19.9 mm to (19.4, 56.8), turned to 90 degrees
- moved R7 19.3 mm to (43.3, 56.7), turned to 0 degrees
- moved R9 19.2 mm to (11.1, 19.6)
- moved R12 17.8 mm to (10.7, 69.9), turned to 180 degrees
- moved R13 15.2 mm to (25.3, 69.9), turned to 180 degrees
- moved R11 15.0 mm to (6.33, 110.9), turned to 0 degrees
- moved R4 14.1 mm to (32.2, 56.7)
- moved R6 13.7 mm to (43.3, 53.0), turned to 0 degrees
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Connections:
- removed net 3BAND_OUT: R12.P$2, R13.P$2, R14.P$2, R8.1
- removed net ATTINY_[PROGRAM_SIGNAL_3: U1.D11, U2.5
- removed net ATTINY_[PROGRAM_SIGNAL_4: U1.D10, U2.1
- removed net N$1: D1.A, R15.1
- removed net N$13: C3.A, L3.P$1, R2.2
- removed net N$14: C4.A, L3.P$2, L4.P$1
- removed net N$15: C5.A, L4.P$2, R10.P$30, R3.1
- removed net N$17: R11.P$3, R8.2, S3.P$2, U3.2
- removed net N$18: C6.C, R12.P$3, R4.1
- removed net N$19: C7.A, R13.P$3, R5.2
- removed net N$20: C8.C, R6.1, R7.1
- removed net N$21: C9.A, R14.P$3, R7.2
- removed net N$26: C6.A, C8.A, R5.1, S3.P$1
- removed net ON_OFF_STATE: R1.2, R15.2, S1.P$3, S1.P$4, U1.D12, U2.6
- removed net VAR_FREQ: R9.P$2, U1.D13, U2.7
- new net AMP_NEG: R11.P$3, R24.2, U3.2
- new net ATTINY_PROGRAM_1: JP4.2, JP6.2, U2.7
- new net ATTINY_PROGRAM_SIGNAL_1: JP1.D13, JP6.1
- new net ATTINY_PROGRAM_SIGNAL_2: JP1.D12, JP7.1
- new net ATTINY_PROGRAM_SIGNAL_3: JP1.D11, JP9.1
- new net ATTINY_PROGRAM_SIGNAL_4: JP1.D10, JP8.1
- new net BPF_ATTENUATED: R14.P$2, R17.1
- new net BPF_INTERMEDIATE: C15.C, R6.1, R7.1
- new net BPF_OUT: C17.A, R14.P$3, R7.2
- new net CHEBYSHEV_IN: JP10.2, R2.1
- new net CHEBYSHEV_STAGE_1: C11.A, L3.P$1, R2.2
- new net CHEBYSHEV_STAGE_2: C12.A, L3.P$2, L4.P$1
- new net CHEBYSHEV_STAGE_3: C13.A, L4.P$2, R29.P$3, R3.1
- new net EQ_IN: C14.A, C15.A, R5.1, SW3.P$1
- new net EQ_OUT: R16.2, R17.2, R8.2, SW3.P$2, U3.3
- new net HPF_ATTENUATED: R12.P$2, R8.1
- new net HPF_OUT: C14.C, R12.P$3, R4.1
- new net LED_POSITIVE: LED1.A, R15.1
- new net LPF_ATTENUATED: R13.P$2, R16.1
- new net LPF_OUT: C16.A, R13.P$3, R5.2
- new net PROGRAM3: JP9.2, U2.5
- new net PROGRAM4: JP8.2, U2.1
- new net SLIDE_SWITCH_IN: JP11.2, SW3.P$3
- new net STATE_SWITCH: JP3.2, JP7.2, U2.6
- new net STATE_SWITCH_OUT: JP3.1, R15.2, SW1.P$2, SW1.P$3
- new net UNO_TONE_MASTER_OUT: JP5.1, R1.1, SW2.5, SW2.6, SW2.7, SW2.8
- new net VAR_FREQ_OUT: JP4.1, R9.P$2
- net +5V: now also C18.A, JP1.5V, SW1.P$1, SW1.P$4; no longer C1.A, C2.A, S1.P$1, S1.P$2, U1.5V
- net CHEBYSHEV_OUT: now also JP11.1, R29.P$2; no longer R10.P$20, S3.P$3
- net DDS_TONE_OUTPUT: now also JP10.1; no longer R2.1
- net GND: now also C11.C, C12.C, C13.C, C16.C, C17.C, C18.C, JP1.GND@0, JP1.GND@1, JP1.GND@2, JP2.2, LED1.C, R1.2, R24.1, R29.P$1; no longer C1.C, C2.C, C3.C, C4.C, C5.C, C7.C, C9.C, D1.C, J1.2, R1.1, R10.P$10, R11.P$1, U1.GND@1, U3.3
- net SPEAKER_IN: now also JP2.1; no longer J1.1
- net UNO_TONE_1: now also JP1.D3, SW2.4; no longer S2.4, U1.D3
- net UNO_TONE_2: now also JP1.D5, SW2.3; no longer S2.3, U1.D5
- net UNO_TONE_3: now also JP1.D6, SW2.2; no longer S2.2, U1.D6
- net UNO_TONE_4: now also JP1.D9, SW2.1; no longer S2.1, U1.D9
- net UNO_TONE_MASTER: now also JP5.2; no longer S2.5, S2.6, S2.7, S2.8
Routing:
- net GND: track 256.7 -> 74.0 mm, vias 3 -> 7
- net N$17: track 117.4 -> 0.00 mm
- net EQ_OUT: track 0.00 -> 107.0 mm, vias 0 -> 3
- net STATE_SWITCH: track 0.00 -> 53.8 mm, vias 0 -> 1
- net ON_OFF_STATE: track 50.6 -> 0.00 mm
- net 3BAND_OUT: track 49.5 -> 0.00 mm
- net HPF_OUT: track 0.00 -> 37.9 mm
- net N$21: track 36.1 -> 0.00 mm
- net N$18: track 34.3 -> 0.00 mm
- net LPF_OUT: track 0.00 -> 30.2 mm
- net EQ_IN: track 0.00 -> 27.8 mm
- net N$15: track 25.3 -> 0.00 mm, vias 1 -> 0
- net AMP_NEG: track 0.00 -> 25.1 mm
- net BPF_OUT: track 0.00 -> 23.7 mm
- net CHEBYSHEV_STAGE_3: track 0.00 -> 21.8 mm
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- added copper zone on layer 16, net GND
Other:
- board size 55.1 x 177.8 mm -> 54.6 x 127 mm
