File: 3 Realization/Eagle/DDS Tone Shield/DDS Tone Shield.sch (EAGLE design)
At the start: 37 parts, among them J1 Speaker Header, U2 ATTINY85-20P, U3 LM386N

Commit message: layout
layout
Parts:
- removed C1, C2, C4: 100nF, DDS Tone Shield:CAP_POL1206
- removed C3, C5: 47nF, DDS Tone Shield:CAP_POL1206
- removed C6, C7, C8, C9: 22nF, DDS Tone Shield:CAP_POL1206
- removed D1: BLUE, DDS Tone Shield:LED-BLUE1206
- removed J1: Speaker Header, DDS Tone Shield:CONN_02
- removed R10: 100kohm, DDS Tone Shield:POT2
- removed S1: PUSHBUTTON, DDS Tone Shield:PUSHBUTTON
- removed S2: DIP-04SMD, DDS Tone Shield:DIP-04SMD
- removed S3: Slide Switch, DDS Tone Shield:SWITCH-SPDT
- added C11, C13: 47nF, 1-Generic:CAP1206
- added C12, C18: 100nF, 1-Generic:CAP1206
- added C14, C15, C16, C17: 22nF, 1-Generic:CAP1206
- added JP10, JP11, JP3, JP4, JP5, JP6, JP7, JP8, JP9: JUMPER-SMT_2_NC_PASTE_SILK, DDS Tone Shield:JUMPER-SMT_2_NC_PASTE_SILK
- added JP2: Speaker Header, DDS Tone Shield:CONN_02
- added LED1: BLUE, DDS Tone Shield:LED-BLUE1206
- added R16, R17: 2200, DDS Tone Shield:RESISTOR1206
- added R24: 270ohm, DDS Tone Shield:RESISTOR1206
- added R29: 100k, DDS Tone Shield:POT1
- added SW1: PUSHBUTTON, DDS Tone Shield:PUSHBUTTON
- added SW2: DIP-04SMD, DDS Tone Shield:DIP-04SMD
- added SW3: Slide Switch, DDS Tone Shield:SWITCH-SPDT
- C10: value (none) -> 100nF; device DDS Tone Shield:CAP_POL1206 -> 1-Generic:CAP1206
- JP1: value (none) -> Arduino jumpers
- R1: value 330ohm -> 10kohm
- R8: value 5.6kohm -> 2200
- Y1: value (none) -> Speaker
- renumbered U1 to JP1
Connections:
- removed net 3BAND_OUT: R12.S, R13.S, R14.S, R8.1
- removed net ATTINY_[PROGRAM_SIGNAL_3: JP1.D11, U2.PB0
- removed net ATTINY_[PROGRAM_SIGNAL_4: JP1.D10, U2.NRES/PB5
- removed net N$1: D1.A, R15.1
- removed net N$13: C3.+, L3.1, R2.2
- removed net N$14: C4.+, L3.2, L4.1
- removed net N$15: C5.+, L4.2, R10.E, R3.1
- removed net N$17: R11.E, R8.2, S3.O, U3.-IN
- removed net N$18: C6.-, R12.E, R4.1
- removed net N$19: C7.+, R13.E, R5.2
- removed net N$20: C8.-, R6.1, R7.1
- removed net N$21: C9.+, R14.E, R7.2
- removed net N$26: C6.+, C8.+, R5.1, S3.S
- removed net ON_OFF_STATE: JP1.D12, R1.2, R15.2, S1.B1, S1.B2, U2.PB1
- removed net VAR_FREQ: JP1.D13, R9.S, U2.PB2
- new net AMP_NEG: R11.E, R24.2, U3.-IN
- new net ATTINY_PROGRAM_1: JP4.2, JP6.2, U2.PB2
- new net ATTINY_PROGRAM_SIGNAL_1: JP1.D13, JP6.1
- new net ATTINY_PROGRAM_SIGNAL_2: JP1.D12, JP7.1
- new net ATTINY_PROGRAM_SIGNAL_3: JP1.D11, JP9.1
- new net ATTINY_PROGRAM_SIGNAL_4: JP1.D10, JP8.1
- new net BPF_ATTENUATED: R14.S, R17.1
- new net BPF_INTERMEDIATE: C15.2, R6.1, R7.1
- new net BPF_OUT: C17.1, R14.E, R7.2
- new net CHEBYSHEV_IN: JP10.2, R2.1
- new net CHEBYSHEV_STAGE_1: C11.1, L3.1, R2.2
- new net CHEBYSHEV_STAGE_2: C12.1, L3.2, L4.1
- new net CHEBYSHEV_STAGE_3: C13.1, L4.2, R29.E, R3.1
- new net EQ_IN: C14.1, C15.1, R5.1, SW3.S
- new net EQ_OUT: R16.2, R17.2, R8.2, SW3.O, U3.+IN
- new net HPF_ATTENUATED: R12.S, R8.1
- new net HPF_OUT: C14.2, R12.E, R4.1
- new net LED_POSITIVE: LED1.A, R15.1
- new net LPF_ATTENUATED: R13.S, R16.1
- new net LPF_OUT: C16.1, R13.E, R5.2
- new net PROGRAM3: JP9.2, U2.PB0
- new net PROGRAM4: JP8.2, U2.NRES/PB5
- new net SLIDE_SWITCH_IN: JP11.2, SW3.P
- new net STATE_SWITCH: JP3.2, JP7.2, U2.PB1
- new net STATE_SWITCH_OUT: JP3.1, R15.2, SW1.A2, SW1.B2
- new net UNO_TONE_MASTER_OUT: JP5.1, R1.1, SW2.1B, SW2.2B, SW2.3B, SW2.4B
- new net VAR_FREQ_OUT: JP4.1, R9.S
- net +5V: now also C10.1, C18.1, SW1.A1, SW1.B1; no longer C1.+, C10.+, C2.+, S1.A1, S1.A2
- net CHEBYSHEV_OUT: now also JP11.1, R29.S; no longer R10.S, S3.P
- net DDS_TONE_OUTPUT: now also JP10.1; no longer R2.1
- net GND: now also C10.2, C11.2, C12.2, C13.2, C16.2, C17.2, C18.2, JP1.GND@0, JP1.GND@2, JP2.2, LED1.C, R1.2, R24.1, R29.A; no longer C1.-, C10.-, C2.-, C3.-, C4.-, C5.-, C7.-, C9.-, D1.C, J1.2, R1.1, R10.A, R11.A, U3.+IN
- net SPEAKER_IN: now also JP2.1; no longer J1.1
- net UNO_TONE_1: now also SW2.4A; no longer S2.4A
- net UNO_TONE_2: now also SW2.3A; no longer S2.3A
- net UNO_TONE_3: now also SW2.2A; no longer S2.2A
- net UNO_TONE_4: now also SW2.1A; no longer S2.1A
- net UNO_TONE_MASTER: now also JP5.2; no longer S2.1B, S2.2B, S2.3B, S2.4B
Other:
- note added: "- Standard Passives - Resistors Standard 1206, .25W, 5% - Capacitors non Standard 1206 , 25V, 20% - Inductors - 4.7mH - 40 mA - 5mm x 5.5mm - LEDs - LTST-C150TBKT - Blue"
- moved on the sheet: R1, R11, R12, R13, R14, R15, R4, R5, R6, R7, R8, R9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
